Commit message: added vacuum gripper

File: src/universal_robot/ur_description/urdf/orig/ur5_joint_limited_robot.urdf.xacro (robot description, xacro)
@@ -1,5 +1,6 @@
 <?xml version="1.0"?>
-<robot xmlns:xacro="http://ros.org/wiki/xacro"
+<robot xmlns:xacro="http://wiki.ros.org/xacro"
        name="ur5" >
+  <xacro:arg name="transmission_hw_interface" default="hardware_interface/PositionJointInterface"/>
   <!-- common stuff -->
   <xacro:include filename="$(find ur_description)/urdf/common.gazebo.xacro" />
@@ -14,4 +15,5 @@
     wrist_2_lower_limit="${-pi}" wrist_2_upper_limit="${pi}"
     wrist_3_lower_limit="${-pi}" wrist_3_upper_limit="${pi}"
+    transmission_hw_interface="$(arg transmission_hw_interface)"
   />
   <link name="world" />

File: src/ur5_t2_4230/ur_description/orig/ur5.urdf.xacro (robot description, xacro)
@@ -12,5 +12,5 @@
   <xacro:property name="wrist_3_mass" value="0.1879" />
   <xacro:property name="height3" value="1" /> <!-- Link 3 -->
-  <xacro:property name="camera_link" value="0.02" /> <!-- Size of square 'camera' box -->
+  <xacro:property name="camera_link" value="0.05" /> <!-- Size of square 'camera' box -->
   <xacro:property name="axel_offset" value="0.05" /> <!-- Space btw top of beam and the each joint -->
   <xacro:property name="shoulder_cog" value="0.0 0.00193 -0.02561" />
@@ -76,7 +76,5 @@
      wrist_1_lower_limit:=${-pi}    wrist_1_upper_limit:=${pi}
      wrist_2_lower_limit:=${-pi}    wrist_2_upper_limit:=${pi}
-     wrist_3_lower_limit:=${-pi}    wrist_3_upper_limit:=${pi}
-    transmission_hw_interface:=hardware_interface/PositionJointInterface"
->
+     wrist_3_lower_limit:=${-pi}    wrist_3_upper_limit:=${pi}">
     <link name="${prefix}base_link" >
       <visual>
@@ -293,369 +291,8 @@
           <box size="0.01 0.01 0.01"/>
         </geometry>
-        <surface>
-          <friction>
-            <ode>
-              <mu>10</mu>
-              <mu2>10</mu2>
-            </ode>
-          </friction>
-        </surface>
         <origin rpy="0 0 0" xyz="-0.01 0 0"/>
       </collision>
     </link>
-    <link name="vacuum_gripper">
-      <gravity>0</gravity>
-      <visual>
-        <origin rpy="0 0 0" xyz="0 0 0"/>
-        <geometry>
-          <cylinder radius="0.005" length="0.01"/>
-        </geometry>
-        <material name="transparent">
-          <color rgba="0 0 0 0"/>
-        </material>
-      </visual>
-      <inertial>
-        <origin rpy="0 0 0" xyz="0.000000 0.000000 0.000000"/>
-        <mass value="0.0001"/>
-        <inertia ixx="1e-08" ixy="0" ixz="0" iyy="1e-08" iyz="0" izz="1e-08"/>
-      </inertial>
-    </link>
-    <joint name="gripper_joint" type="revolute">
-      <axis xyz="1 0 0" />
-      <parent link="ee_link" />
-      <child link="vacuum_gripper" />
-      <origin rpy="0 1.5708 0" xyz="0.01 0.0125 0" />
-      <limit effort="50" velocity="50" lower="0" upper="0" />
-      <dynamics damping="0.0" friction="10"/>
-    </joint>
-  <gazebo>
-      <plugin name="gazebo_ros_vacuum_gripper" filename="libgazebo_ros_vacuum_gripper.so">
-        <robotNamespace>/ur5/vacuum_gripper</robotNamespace>
-        <bodyName>vacuum_gripper</bodyName>
-        <topicName>grasping</topicName>
-	<maxForce>50</maxForce>
-        <maxDistance>0.05</maxDistance>
-        <minDistance>0.01</minDistance>
-      </plugin>
-  </gazebo>
-    <link name="vacuum_gripper1">
-      <gravity>0</gravity>
-      <visual>
-        <origin rpy="0 0 0" xyz="0 0 0"/>
-        <geometry>
-          <cylinder radius="0.005" length="0.01"/>
-        </geometry>
-        <material name="transparent">
-          <color rgba="0 0 0 0"/>
-        </material>
-      </visual>
-      <inertial>
-        <origin rpy="0 0 0" xyz="0.000000 0.000000 0.000000"/>
-        <mass value="0.0001"/>
-        <inertia ixx="1e-08" ixy="0" ixz="0" iyy="1e-08" iyz="0" izz="1e-08"/>
-      </inertial>
-    </link>
-    <joint name="gripper_joint1" type="revolute">
-      <axis xyz="1 0 0" />
-      <parent link="ee_link" />
-      <child link="vacuum_gripper1" />
-      <origin rpy="0 1.5708 0" xyz="0.01 -0.0125 0" />
-      <limit effort="50" velocity="50" lower="0" upper="0" />
-      <dynamics damping="0.0" friction="10"/>
-    </joint>
-  <gazebo>
-      <plugin name="gazebo_ros_vacuum_gripper1" filename="libgazebo_ros_vacuum_gripper.so">
-        <robotNamespace>/ur5/vacuum_gripper1</robotNamespace>
-        <bodyName>vacuum_gripper1</bodyName>
-        <topicName>grasping1</topicName>
-	<maxForce>50</maxForce>
-        <maxDistance>0.05</maxDistance>
-        <minDistance>0.01</minDistance>
-      </plugin>
-  </gazebo>
-    <link name="vacuum_gripper2">
-      <gravity>0</gravity>
-      <visual>
-        <origin rpy="0 0 0" xyz="0 0 0"/>
-        <geometry>
-          <cylinder radius="0.005" length="0.01"/>
-        </geometry>
-        <material name="transparent">
-          <color rgba="0 0 0 0"/>
-        </material>
-      </visual>
-      <inertial>
-        <origin rpy="0 0 0" xyz="0.000000 0.000000 0.000000"/>
-        <mass value="0.0001"/>
-        <inertia ixx="1e-08" ixy="0" ixz="0" iyy="1e-08" iyz="0" izz="1e-08"/>
-      </inertial>
-    </link>
-    <joint name="gripper_joint2" type="revolute">
-      <axis xyz="1 0 0" />
-      <parent link="ee_link" />
-      <child link="vacuum_gripper2" />
-      <origin rpy="0 1.5708 0" xyz="0.01 0 0.0125" />
-      <limit effort="50" velocity="50" lower="0" upper="0" />
-      <dynamics damping="0.0" friction="10"/>
-    </joint>
-  <gazebo>
-      <plugin name="gazebo_ros_vacuum_gripper2" filename="libgazebo_ros_vacuum_gripper.so">
-        <robotNamespace>/ur5/vacuum_gripper2</robotNamespace>
-        <bodyName>vacuum_gripper2</bodyName>
-        <topicName>grasping2</topicName>
-	<maxForce>50</maxForce>
-        <maxDistance>0.05</maxDistance>
-        <minDistance>0.01</minDistance>
-      </plugin>
-  </gazebo>
-    <link name="vacuum_gripper3">
-      <gravity>0</gravity>
-      <visual>
-        <origin rpy="0 0 0" xyz="0 0 0"/>
-        <geometry>
-          <cylinder radius="0.005" length="0.01"/>
-        </geometry>
-        <material name="transparent">
-          <color rgba="0 0 0 0"/>
-        </material>
-      </visual>
-      <inertial>
-        <origin rpy="0 0 0" xyz="0.000000 0.000000 0.000000"/>
-        <mass value="0.0001"/>
-        <inertia ixx="1e-08" ixy="0" ixz="0" iyy="1e-08" iyz="0" izz="1e-08"/>
-      </inertial>
-    </link>
-    <joint name="gripper_joint3" type="revolute">
-      <axis xyz="1 0 0" />
-      <parent link="ee_link" />
-      <child link="vacuum_gripper3" />
-      <origin rpy="0 1.5708 0" xyz="0.01 0 -0.0125" />
-      <limit effort="50" velocity="50" lower="0" upper="0" />
-      <dynamics damping="0.0" friction="10"/>
-    </joint>
-  <gazebo>
-      <plugin name="gazebo_ros_vacuum_gripper3" filename="libgazebo_ros_vacuum_gripper.so">
-        <robotNamespace>/ur5/vacuum_gripper3</robotNamespace>
-        <bodyName>vacuum_gripper3</bodyName>
-        <topicName>grasping2</topicName>
-	<maxForce>50</maxForce>
-        <maxDistance>0.05</maxDistance>
-        <minDistance>0.01</minDistance>
-      </plugin>
-  </gazebo>
-  <link name="vacuum_gripper4">
-    <gravity>0</gravity>
-    <visual>
-      <origin rpy="0 0 0" xyz="0 0 0"/>
-      <geometry>
-        <cylinder radius="0.005" length="0.01"/>
-      </geometry>
-      <material name="transparent">
-        <color rgba="0 0 0 0"/>
-      </material>
-    </visual>
-    <inertial>
-      <origin rpy="0 0 0" xyz="0.000000 0.000000 0.000000"/>
-      <mass value="0.0001"/>
-      <inertia ixx="1e-08" ixy="0" ixz="0" iyy="1e-08" iyz="0" izz="1e-08"/>
-    </inertial>
-  </link>
-  <joint name="gripper_joint4" type="revolute">
-    <axis xyz="1 0 0" />
-    <parent link="ee_link" />
-    <child link="vacuum_gripper4" />
-    <origin rpy="0 1.5708 0" xyz="0.01 0 0" />
-    <limit effort="50" velocity="50" lower="0" upper="0" />
-    <dynamics damping="0.0" friction="10"/>
-  </joint>
-  <gazebo>
-    <plugin name="gazebo_ros_vacuum_gripper4" filename="libgazebo_ros_vacuum_gripper.so">
-      <robotNamespace>/ur5/vacuum_gripper4</robotNamespace>
-      <bodyName>vacuum_gripper4</bodyName>
-      <topicName>grasping4</topicName>
-  <maxForce>50</maxForce>
-      <maxDistance>0.05</maxDistance>
-      <minDistance>0.01</minDistance>
-    </plugin>
-  </gazebo>
-  <link name="vacuum_gripper5">
-    <gravity>0</gravity>
-    <visual>
-      <origin rpy="0 0 0" xyz="0 0 0"/>
-      <geometry>
-        <cylinder radius="0.005" length="0.01"/>
-      </geometry>
-      <material name="transparent">
-        <color rgba="0 0 0 0"/>
-      </material>
-    </visual>
-    <inertial>
-      <origin rpy="0 0 0" xyz="0.000000 0.000000 0.000000"/>
-      <mass value="0.0001"/>
-      <inertia ixx="1e-08" ixy="0" ixz="0" iyy="1e-08" iyz="0" izz="1e-08"/>
-    </inertial>
-  </link>
-  <joint name="gripper_joint5" type="revolute">
-    <axis xyz="1 0 0" />
-    <parent link="ee_link" />
-    <child link="vacuum_gripper5" />
-    <origin rpy="0 1.5708 0" xyz="0.01 0.0125 0.0125" />
-    <limit effort="50" velocity="50" lower="0" upper="0" />
-    <dynamics damping="0.0" friction="10"/>
-  </joint>
-<gazebo>
-    <plugin name="gazebo_ros_vacuum_gripper" filename="libgazebo_ros_vacuum_gripper.so">
-      <robotNamespace>/ur5/vacuum_gripper5</robotNamespace>
-      <bodyName>vacuum_gripper5</bodyName>
-      <topicName>grasping5</topicName>
-<maxForce>50</maxForce>
-      <maxDistance>0.05</maxDistance>
-      <minDistance>0.01</minDistance>
-    </plugin>
-</gazebo>
-  <link name="vacuum_gripper6">
-    <gravity>0</gravity>
-    <visual>
-      <origin rpy="0 0 0" xyz="0 0 0"/>
-      <geometry>
-        <cylinder radius="0.005" length="0.01"/>
-      </geometry>
-      <material name="transparent">
-        <color rgba="0 0 0 0"/>
-      </material>
-    </visual>
-    <inertial>
-      <origin rpy="0 0 0" xyz="0.000000 0.000000 0.000000"/>
-      <mass value="0.0001"/>
-      <inertia ixx="1e-08" ixy="0" ixz="0" iyy="1e-08" iyz="0" izz="1e-08"/>
-    </inertial>
-  </link>
-  <joint name="gripper_joint6" type="revolute">
-    <axis xyz="1 0 0" />
-    <parent link="ee_link" />
-    <child link="vacuum_gripper6" />
-    <origin rpy="0 1.5708 0" xyz="0.01 -0.0125 0.0125" />
-    <limit effort="50" velocity="50" lower="0" upper="0" />
-    <dynamics damping="0.0" friction="10"/>
-  </joint>
-<gazebo>
-    <plugin name="gazebo_ros_vacuum_gripper1" filename="libgazebo_ros_vacuum_gripper.so">
-      <robotNamespace>/ur5/vacuum_gripper6</robotNamespace>
-      <bodyName>vacuum_gripper6</bodyName>
-      <topicName>grasping6</topicName>
-<maxForce>50</maxForce>
-      <maxDistance>0.05</maxDistance>
-      <minDistance>0.01</minDistance>
-    </plugin>
-</gazebo>
-  <link name="vacuum_gripper7">
-    <gravity>0</gravity>
-    <visual>
-      <origin rpy="0 0 0" xyz="0 0 0"/>
-      <geometry>
-        <cylinder radius="0.005" length="0.01"/>
-      </geometry>
-      <material name="transparent">
-        <color rgba="0 0 0 0"/>
-      </material>
-    </visual>
-    <inertial>
-      <origin rpy="0 0 0" xyz="0.000000 0.000000 0.000000"/>
-      <mass value="0.0001"/>
-      <inertia ixx="1e-08" ixy="0" ixz="0" iyy="1e-08" iyz="0" izz="1e-08"/>
-    </inertial>
-  </link>
-  <joint name="gripper_joint7" type="revolute">
-    <axis xyz="1 0 0" />
-    <parent link="ee_link" />
-    <child link="vacuum_gripper7" />
-    <origin rpy="0 1.5708 0" xyz="0.01 0.0125 -0.0125" />
-    <limit effort="50" velocity="50" lower="0" upper="0" />
-    <dynamics damping="0.0" friction="10"/>
-  </joint>
-<gazebo>
-    <plugin name="gazebo_ros_vacuum_gripper7" filename="libgazebo_ros_vacuum_gripper.so">
-      <robotNamespace>/ur5/vacuum_gripper7</robotNamespace>
-      <bodyName>vacuum_gripper7</bodyName>
-      <topicName>grasping7</topicName>
-<maxForce>50</maxForce>
-      <maxDistance>0.05</maxDistance>
-      <minDistance>0.01</minDistance>
-    </plugin>
-</gazebo>
-  <link name="vacuum_gripper8">
-    <gravity>0</gravity>
-    <visual>
-      <origin rpy="0 0 0" xyz="0 0 0"/>
-      <geometry>
-        <cylinder radius="0.005" length="0.01"/>
-      </geometry>
-      <material name="transparent">
-        <color rgba="0 0 0 0"/>
-      </material>
-    </visual>
-    <inertial>
-      <origin rpy="0 0 0" xyz="0.000000 0.000000 0.000000"/>
-      <mass value="0.0001"/>
-      <inertia ixx="1e-08" ixy="0" ixz="0" iyy="1e-08" iyz="0" izz="1e-08"/>
-    </inertial>
-  </link>
-  <joint name="gripper_joint8" type="revolute">
-    <axis xyz="1 0 0" />
-    <parent link="ee_link" />
-    <child link="vacuum_gripper8" />
-    <origin rpy="0 1.5708 0" xyz="0.01 -0.0125 -0.0125" />
-    <limit effort="50" velocity="50" lower="0" upper="0" />
-    <dynamics damping="0.0" friction="10"/>
-  </joint>
-<gazebo>
-    <plugin name="gazebo_ros_vacuum_gripper8" filename="libgazebo_ros_vacuum_gripper.so">
-      <robotNamespace>/ur5/vacuum_gripper8</robotNamespace>
-      <bodyName>vacuum_gripper8</bodyName>
-      <topicName>grasping8</topicName>
-<maxForce>50</maxForce>
-      <maxDistance>0.05</maxDistance>
-      <minDistance>0.01</minDistance>
-    </plugin>
-</gazebo>
-  <joint name="camera_joint" type="fixed">
-    <axis xyz="0 1 0" />
-    <origin xyz="-0.02 0.0 0.055" rpy="0 0 0"/>
-    <parent link="ee_link"/>
-    <child link="camera_link"/>
-  </joint>
-  <!-- Camera -->
-  <link name="camera_link">
-    <collision>
-      <origin xyz="0 0 0" rpy="0 0 0"/>
-      <geometry>
-	<box size="${camera_link} ${camera_link} ${camera_link}"/>
-      </geometry>
-    </collision>
-    <visual>
-      <origin xyz="0 0 0" rpy="0 0 0"/>
-      <geometry>
-	<box size="${camera_link} ${camera_link} ${camera_link}"/>
-      </geometry>
-      <material name="green"/>
-    </visual>
-    <inertial>
-      <mass value="1e-5" />
-      <origin xyz="0 0 0" rpy="0 0 0"/>
-      <inertia ixx="1e-6" ixy="0" ixz="0" iyy="1e-6" iyz="0" izz="1e-6" />
-    </inertial>
-  </link>
-  <!-- generate an optical frame http://www.ros.org/reps/rep-0103.html#suffix-frames
-      so that ros and opencv can operate on the camera frame correctly -->
-  <joint name="camera_optical_joint" type="fixed">
-    <!-- these values have to be these values otherwise the gazebo camera image
-        won't be aligned properly with the frame it is supposedly originating from -->
-    <origin xyz="0 0 0" rpy="${-pi/2} 0 ${-pi/2}"/>
-    <parent link="camera_link"/>
-    <child link="camera_link_optical"/>
-  </joint>
-  <link name="camera_link_optical">
-  </link>
-    <xacro:ur_arm_transmission prefix="${prefix}" hw_interface="${transmission_hw_interface}"/>
+    <xacro:ur_arm_transmission prefix="${prefix}" />
     <xacro:ur_arm_gazebo prefix="${prefix}" />
     <!-- ROS base_link to UR 'Base' Coordinates transform -->

File: src/ur5_t2_4230/ur_description/ur5.urdf.xacro (robot description, xacro)
@@ -76,7 +76,5 @@
      wrist_1_lower_limit:=${-pi}    wrist_1_upper_limit:=${pi}
      wrist_2_lower_limit:=${-pi}    wrist_2_upper_limit:=${pi}
-     wrist_3_lower_limit:=${-pi}    wrist_3_upper_limit:=${pi}
-    transmission_hw_interface:=hardware_interface/PositionJointInterface"
->
+     wrist_3_lower_limit:=${-pi}    wrist_3_upper_limit:=${pi}">
     <link name="${prefix}base_link" >
       <visual>
@@ -657,5 +655,5 @@
   <link name="camera_link_optical">
   </link>
-    <xacro:ur_arm_transmission prefix="${prefix}" hw_interface="${transmission_hw_interface}"/>
+    <xacro:ur_arm_transmission prefix="${prefix}" />
     <xacro:ur_arm_gazebo prefix="${prefix}" />
     <!-- ROS base_link to UR 'Base' Coordinates transform -->

File: src/ur5_t2_4230/ur_description/ur5_joint_limited_robot.urdf.xacro (robot description, xacro)
@@ -8,5 +8,5 @@
   <!-- arm -->
   <xacro:ur5_robot prefix="" joint_limited="true"
-    shoulder_pan_lower_limit="${-pi}" shoulder_pan_upper_limit="${pi}"
+    shoulder_pan_lower_limit="${-2*pi}" shoulder_pan_upper_limit="${2*pi}"
     shoulder_lift_lower_limit="${-pi}" shoulder_lift_upper_limit="${pi}"
     elbow_joint_lower_limit="${-pi}" elbow_joint_upper_limit="${pi}"
