Commit message: sometimes suckable

File: src/ur5_t2_4230/models/red_box.urdf (robot description, URDF)
Before this commit: robot red_box, 1 links, 0 joints
Links:
- link base_link: mass 0.05 -> 0.5; geometry collision box size=0.1 0.075 0.05; visual box size=0.1 0.075 0.05

Commit message: update git ignore and physics shit

File: src/ur5_t2_4230/models/red_box.urdf (robot description, URDF)
Before this commit: robot red_box, 1 links, 0 joints
Links:
- link base_link: mass 0.5 -> 0.6

Commit message: consistently 90

File: src/ur5_t2_4230/models/red_box.urdf (robot description, URDF)
Before this commit: robot red_box, 1 links, 0 joints
Links:
- link base_link: mass 0.6 -> 0.01
