Commit message: complete; todo: clean up code

File: src/universal_robot/ur_description/urdf/ur5.urdf.xacro (robot description, xacro)
@@ -633,5 +633,5 @@
       </geometry>
     </collision>
-    <visual>
+    <!-- <visual>
       <origin xyz="0 0 0" rpy="0 0 0"/>
       <geometry>
@@ -639,5 +639,5 @@
       </geometry>
       <material name="green"/>
-    </visual>
+    </visual> -->
     <inertial>
       <mass value="1e-5" />

File: src/ur5_t2_4230/models/blue_box.urdf (robot description, URDF)
Before this commit: robot red_box, 1 links, 0 joints
Links:
- link base_link: geometry collision box size=0.075 0.075 0.05; visual box size=0.075 0.075 0.05

File: src/ur5_t2_4230/models/blue_cylinder.urdf (robot description, URDF)
Before this commit: robot blue_cylinder, 1 links, 0 joints
Links:
- link base_link: geometry collision cylinder length=0.05 radius=0.0375; visual cylinder length=0.05 radius=0.0375

File: src/ur5_t2_4230/models/green_box.urdf (robot description, URDF)
Before this commit: robot red_box, 1 links, 0 joints
Links:
- link base_link: geometry collision box size=0.075 0.075 0.05; visual box size=0.075 0.075 0.05

File: src/ur5_t2_4230/models/green_cylinder.urdf (robot description, URDF)
Before this commit: robot green_cylinder, 1 links, 0 joints
Links:
- link base_link: geometry collision cylinder length=0.05 radius=0.0375; visual cylinder length=0.05 radius=0.0375

File: src/ur5_t2_4230/models/red_box.urdf (robot description, URDF)
Before this commit: robot red_box, 1 links, 0 joints
Links:
- link base_link: geometry collision box size=0.075 0.075 0.05; visual box size=0.075 0.075 0.05

File: src/ur5_t2_4230/models/red_cylinder.urdf (robot description, URDF)
Before this commit: robot red_cylinder, 1 links, 0 joints
Links:
- link base_link: geometry collision cylinder length=0.05 radius=0.0375; visual cylinder length=0.05 radius=0.0375
